File: common-cathode/LED_port-status-CC.kicad_pcb (KiCad board)
At the start: 2 copper layers, 23.7 x 9 mm, 13 parts, among them P1 CONN_9

Commit message: CA / CC tweaks.
Other:
- board text removed: "-"
Changed lines of the file:
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@@
     (area 79.31 84.07974 103.404433 93.267601)
     (thickness 1.6)
-    (drawings 16)
+    (drawings 14)
     (tracks 67)
     (zones 0)
@@
   (gr_circle (center 80.01 92.71) (end 80.0354 92.71) (layer Dwgs.User) (width 0.02))
   (gr_circle (center 80.01 84.709) (end 80.0354 84.709) (layer Dwgs.User) (width 0.02))
-  (gr_text - (at 101.6 88.6968) (layer F.SilkS)
-    (effects (font (size 2 2) (thickness 0.3)))
-  )
-  (gr_text - (at 101.6 88.6968) (layer B.SilkS)
-    (effects (font (size 2 2) (thickness 0.3)) (justify mirror))
-  )
   (gr_text 2013 (at 81.8388 85.4456) (layer B.SilkS)
     (effects (font (size 1 1) (thickness 0.2)) (justify mirror))
@@
       )
     )
+  )
+  (zone (net 0) (net_name "") (layer F.Mask) (hatch full 0.508)
+    (connect_pads (clearance 0.2))
+    (min_thickness 0.254)
+    (fill (arc_segments 16) (thermal_gap 0.508) (thermal_bridge_width 0.508))
+    (polygon
+      (pts
+        (xy 100.4824 89.8398) (xy 100.4824 87.7824) (xy 102.7176 87.7824) (xy 102.7176 89.8398)
+      )
+    )
+  )
+  (zone (net 0) (net_name "") (layer B.Mask) (hatch full 0.508)
+    (connect_pads (clearance 0.2))
+    (min_thickness 0.254)
+    (fill (arc_segments 16) (thermal_gap 0.508) (thermal_bridge_width 0.508))
+    (polygon
+      (pts
+        (xy 100.4824 89.8398) (xy 100.4824 87.7824) (xy 102.7176 87.7824) (xy 102.7176 89.8398)
+      )
+    )
